Commit message: setup right arm

File: urdf/material.xacro (robot description, xacro)
@@ -2,4 +2,5 @@
 <!-- material macro for visual color of the robot-->
 <robot name="separable_jaws" xmlns:xacro="http://www.ros.org/wiki/xacro">
+    <!-- material for urdf visual -->
     <material name="Red">
         <color rgba="${204/255} ${0/255} ${0/255} 1.0"/>
@@ -14,4 +15,7 @@
         <color rgba="${255/255} ${255/255} ${255/255} 1.0"/>
     </material>
+    <material name="Light_grey">
+        <color rgba="${204/255} ${204/255} ${204/255} 1.0"/>
+    </material>
     <material name="Grey">
         <color rgba="${100/255} ${100/255} ${100/255} 1.0"/>

File: urdf/separable_jaws.xacro (robot description, xacro)
@@ -1,51 +1,16 @@
 <?xml version="1.0"?>
 <robot name="separable_jaws" xmlns:xacro="http://www.ros.org/wiki/xacro">
-    <!-- include macro from other files-->
+    <!-- include macros from other files-->
     <xacro:include filename="$(find separable_jaws_description)/urdf/material.xacro"/>
     <xacro:include filename="$(find separable_jaws_description)/urdf/simple_geometry.xacro"/>
-    <!-- chassis macro -->
-    <xacro:macro name="chassis" params="name">
-        <xacro:cuboid name="${name}" length="1" width="0.5" hight="0.2" mass="1" material="Red"/>
-    </xacro:macro>
-    <!-- wheel macro -->
-    <xacro:macro name="wheel" params="name">
-        <xacro:cylinder name="${name}" length="0.1" radius="0.3" rpy="${radians(90)} 0 0" mass="1.0" material="Black"/>
-    </xacro:macro>
+    <xacro:include filename="$(find separable_jaws_description)/urdf/parts.xacro"/>
+    <xacro:include filename="$(find separable_jaws_description)/urdf/subassemblies.xacro"/>
     <!-- robot definition -->
-    <link name="base_link">
-    </link>
-    <xacro:chassis name="chassis"/>
-    <xacro:wheel name="front_left_wheel"/>
-    <xacro:wheel name="front_right_wheel"/>
-    <xacro:wheel name="rear_left_wheel"/>
-    <xacro:wheel name="rear_right_wheel"/>
-    <joint name="base_link" type="fixed">
-        <parent link="base_link"/>
-        <child link="chassis"/>
-        <origin xyz="0 0 0.3" rpy="0 0 0"/>
-    </joint>
-    <joint name="front_left_wheel_joint" type="continuous">
-        <parent link="chassis"/>
-        <child link="front_left_wheel"/>
-        <origin xyz="0.4 -0.3 0" rpy="0 0 0"/>
-        <axis xyz="0 1 0"/>
-    </joint>
-    <joint name="front_right_wheel_joint" type="continuous">
-        <parent link="chassis"/>
-        <child link="front_right_wheel"/>
-        <origin xyz="0.4 0.3 0" rpy="0 0 0"/>
-        <axis xyz="0 1 0"/>
-    </joint>
-    <joint name="rear_left_wheel_joint" type="continuous">
-        <parent link="chassis"/>
-        <child link="rear_left_wheel"/>
-        <origin xyz="-0.4 -0.3 0" rpy="0 0 0"/>
-        <axis xyz="0 1 0"/>
-    </joint>
-    <joint name="rear_right_wheel_joint" type="continuous">
-        <parent link="chassis"/>
-        <child link="rear_right_wheel"/>
-        <origin xyz="-0.4 0.3 0" rpy="0 0 0"/>
-        <axis xyz="0 1 0"/>
-    </joint>
+    <link name="base_link"/>
+    <xacro:right_bracket xyz="0 0 1"/>
+    <xacro:right_shoulder/>
+    <xacro:right_upper_arm/>
+    <xacro:right_lower_arm/>
+    <xacro:right_wrist/>
+    <xacro:right_palm/>
 </robot>

File: urdf/simple_geometry.xacro (robot description, xacro)
@@ -4,21 +4,18 @@
     <!-- constant definition -->
     <xacro:property name="triple_zero" value="0 0 0"/>
-    <!-- solid cuboid property macro -->
-    <xacro:macro name="cuboid" params="name length width hight rpy:=${triple_zero} mass material">
+    <!-- solid cuboid property macro, default orientation is length in x-axis, width in y-axis, hight in z-axis -->
+    <xacro:macro name="cuboid" params="name length width hight xyz:=${triple_zero} rpy:=${triple_zero} mass material">
         <link name="${name}">
             <inertial>
-                <origin xyz="0 0 0" rpy="${rpy}"/>
+                <origin xyz="${xyz}" rpy="${rpy}"/>
                 <mass value="${mass}"/>
                 <inertia
-                    ixx="${1 / 12 * mass * (width ** 2 + hight ** 2)}"
-                    iyy="${1 / 12 * mass * (length ** 2 + hight ** 2)}"
+                    ixx="${1 / 12 * mass * (width ** 2 + hight ** 2)}" ixy="0.0" ixz="0.0"
+                    iyy="${1 / 12 * mass * (length ** 2 + hight ** 2)}" iyz="0.0"
                     izz="${1 / 12 * mass * (length ** 2 + width ** 2)}"
-                    ixy="0.0"
-                    ixz="0.0"
-                    iyz="0.0"
                 />
             </inertial>
             <visual>
-                <origin xyz="0 0 0" rpy="${rpy}"/>
+                <origin xyz="${xyz}" rpy="${rpy}"/>
                 <geometry>
                     <box size="${length} ${width} ${hight}"/>
@@ -27,5 +24,5 @@
             </visual>
             <collision>
-                <origin xyz="0 0 0" rpy="${rpy}"/>
+                <origin xyz="${xyz}" rpy="${rpy}"/>
                 <geometry>
                     <box size="${length} ${width} ${hight}"/>
@@ -33,28 +30,22 @@
             </collision>
         </link>
-        <!-- attibutes specfic to gazebo -->
-        <xacro:if value="$(arg using_gazebo)">
-            <gazebo reference="${name}">
-                <material>Gazebo/${material}</material>
-            </gazebo>
-        </xacro:if>
+        <gazebo reference="${name}">
+            <material>Gazebo/${material}</material>
+        </gazebo>
     </xacro:macro>
-    <!-- solid cylinder property macro -->
-    <xacro:macro name="cylinder" params="name length radius rpy:=${triple_zero} mass material">
+    <!-- solid cylinder property macro, default orientation is length in z-axis -->
+    <xacro:macro name="cylinder" params="name length radius xyz:=${triple_zero} rpy:=${triple_zero} mass material">
         <link name="${name}">
             <inertial>
-                <origin xyz="0 0 0" rpy="${rpy}"/>
+                <origin xyz="${xyz}" rpy="${rpy}"/>
                 <mass value="${mass}"/>
                 <inertia
-                    ixx="${1 / 12 * mass * (3 * radius ** 2 + length ** 2)}"
-                    iyy="${1 / 12 * mass * (3 * radius ** 2 + length ** 2)}"
+                    ixx="${1 / 12 * mass * (3 * radius ** 2 + length ** 2)}" ixy="0.0" ixz="0.0"
+                    iyy="${1 / 12 * mass * (3 * radius ** 2 + length ** 2)}" iyz="0.0"
                     izz="${1 / 2 * mass * radius ** 2}"
-                    ixy="0.0"
-                    ixz="0.0"
-                    iyz="0.0"
                 />
             </inertial>
             <visual>
-                <origin xyz="0 0 0" rpy="${rpy}"/>
+                <origin xyz="${xyz}" rpy="${rpy}"/>
                 <geometry>
                     <cylinder length="${length}" radius="${radius}"/>
@@ -63,5 +54,5 @@
             </visual>
             <collision>
-                <origin xyz="0 0 0" rpy="${rpy}"/>
+                <origin xyz="${xyz}" rpy="${rpy}"/>
                 <geometry>
                     <cylinder length="${length}" radius="${radius}"/>
@@ -70,27 +61,22 @@
         </link>
         <!-- attibutes specfic to gazebo -->
-        <xacro:if value="$(arg using_gazebo)">
-            <gazebo reference="${name}">
-                <material>Gazebo/${material}</material>
-            </gazebo>
-        </xacro:if>
+        <gazebo reference="${name}">
+            <material>Gazebo/${material}</material>
+        </gazebo>
     </xacro:macro>
     <!-- solid sphere property macro -->
-    <xacro:macro name="sphere" params="name radius mass material">
+    <xacro:macro name="sphere" params="name radius xyz:=${triple_zero} mass material">
         <link name="${name}">
             <inertial>
-                <origin xyz="0 0 0" rpy="0 0 0"/>
+                <origin xyz="${xyz}" rpy="0 0 0"/>
                 <mass value="${mass}"/>
                 <inertia
-                    ixx="${2 / 5 * mass * radius ** 2}"
-                    iyy="${2 / 5 * mass * radius ** 2}"
+                    ixx="${2 / 5 * mass * radius ** 2}" ixy="0.0" ixz="0.0"
+                    iyy="${2 / 5 * mass * radius ** 2}" iyz="0.0"
                     izz="${2 / 5 * mass * radius ** 2}"
-                    ixy="0.0"
-                    ixz="0.0"
-                    iyz="0.0"
                 />
             </inertial>
             <visual>
-                <origin xyz="0 0 0" rpy="0 0 0"/>
+                <origin xyz="${xyz}" rpy="0 0 0"/>
                 <geometry>
                     <sphere radius="${radius}"/>
@@ -99,5 +85,5 @@
             </visual>
             <collision>
-                <origin xyz="0 0 0" rpy="0 0 0"/>
+                <origin xyz="${xyz}" rpy="0 0 0"/>
                 <geometry>
                     <sphere radius="${radius}"/>
@@ -105,10 +91,7 @@
             </collision>
         </link>
-        <!-- attibutes specfic to gazebo -->
-        <xacro:if value="$(arg using_gazebo)">
-            <gazebo reference="${name}">
-                <material>Gazebo/${material}</material>
-            </gazebo>
-        </xacro:if>
+        <gazebo reference="${name}">
+            <material>Gazebo/${material}</material>
+        </gazebo>
     </xacro:macro>
 </robot>
