Commit message: added left arm

File: urdf/separable_jaws.xacro (robot description, xacro)
@@ -3,10 +3,10 @@
     <!-- include macros from other files-->
     <xacro:include filename="$(find separable_jaws_description)/urdf/material.xacro"/>
-    <xacro:include filename="$(find separable_jaws_description)/urdf/simple_geometry.xacro"/>
     <xacro:include filename="$(find separable_jaws_description)/urdf/parts.xacro"/>
     <xacro:include filename="$(find separable_jaws_description)/urdf/subassemblies.xacro"/>
+    <xacro:include filename="$(find separable_jaws_description)/urdf/ros2_control.xacro"/>
     <!-- robot definition -->
     <link name="base_link"/>
-    <xacro:right_bracket xyz="0 0 1"/>
+    <xacro:right_bracket xyz="0 -0.05 0"/>
     <xacro:right_shoulder/>
     <xacro:right_upper_arm/>
@@ -14,3 +14,10 @@
     <xacro:right_wrist/>
     <xacro:right_palm/>
+    <xacro:left_bracket xyz="0 0.05 0"/>
+    <xacro:left_shoulder/>
+    <xacro:left_upper_arm/>
+    <xacro:left_lower_arm/>
+    <xacro:left_wrist/>
+    <xacro:left_palm/>
+    <xacro:separable_jaws_ros2_control/>
 </robot>

File: urdf/subassemblies.xacro (robot description, xacro)
@@ -1,4 +1,4 @@
 <?xml version="1.0"?>
-<!-- urdf macro inertial, visual and collision for robot parts -->
+<!-- urdf macro attached subassemblies constructed from parts -->
 <robot name="separable_jaws" xmlns:xacro="http://www.ros.org/wiki/xacro">
     <!-- constant definition -->
@@ -7,11 +7,20 @@
     <xacro:include filename="$(find separable_jaws_description)/urdf/parts.xacro"/>
     <!-- subassemblies -->
-    <!-- bracket -->
+    <!-- right_bracket -->
     <xacro:macro name="right_bracket" params="xyz:=${triple_zero}">
         <xacro:bracket name="right_bracket"/>
-        <joint name="mount_point" type="fixed">
+        <joint name="right_mount_point" type="fixed">
             <origin xyz="${xyz}" rpy="0 0 0"/>
             <parent link="base_link"/>
             <child link="right_bracket"/>
+        </joint>
+    </xacro:macro>
+    <!-- left_bracket -->
+    <xacro:macro name="left_bracket" params="xyz:=${triple_zero}">
+        <xacro:bracket name="left_bracket"/>
+        <joint name="left_mount_point" type="fixed">
+            <origin xyz="${xyz}" rpy="${radians(180)} 0 0"/>
+            <parent link="base_link"/>
+            <child link="left_bracket"/>
         </joint>
     </xacro:macro>
@@ -27,7 +36,23 @@
         </joint>
         <joint name="right_shoulder_internal_mount" type="fixed">
-            <origin xyz="0 -0.00005 0" rpy="0 0 0"/>
+            <origin xyz="0 -0.00005 0" rpy="0 ${radians(-90)} 0"/>
             <parent link="right_shoulder_motor"/>
             <child link="right_shoulder"/>
+        </joint>
+    </xacro:macro>
+    <!-- left_shoulder -->
+    <xacro:macro name="left_shoulder">
+        <xacro:dynamixel_pro_h54-100-s500 name="left_shoulder_motor" rpy="0 ${radians(-90)} 0"/>
+        <xacro:shoulder name="left_shoulder"/>
+        <joint name="left_shoulder_joint" type="continuous">
+            <origin xyz="0 -0.025 0" rpy="0 ${radians(180)} 0"/>
+            <parent link="left_bracket"/>
+            <child link="left_shoulder_motor"/>
+            <axis xyz="0 -1 0"/>
+        </joint>
+        <joint name="left_shoulder_internal_mount" type="fixed">
+            <origin xyz="0 -0.00005 0" rpy="0 ${radians(-90)} 0"/>
+            <parent link="left_shoulder_motor"/>
+            <child link="left_shoulder"/>
         </joint>
     </xacro:macro>
@@ -38,5 +63,5 @@
         <xacro:dynamixel_pro_h54-100-s500 name="right_upper_arm_motor2" rpy="0 ${radians(90)} ${radians(90)}"/>
         <joint name="right_upper_arm_joint" type="continuous">
-            <origin xyz="0.045 -0.0505 0" rpy="0 0 0"/>
+            <origin xyz="0.045 -0.0505 0" rpy="${radians(90)} 0 0"/>
             <parent link="right_shoulder"/>
             <child link="right_upper_arm_motor1"/>
@@ -52,4 +77,26 @@
             <parent link="right_upper_arm"/>
             <child link="right_upper_arm_motor2"/>
+        </joint>
+    </xacro:macro>
+    <!-- left_upper_arm -->
+    <xacro:macro name="left_upper_arm">
+        <xacro:dynamixel_pro_h54-200-s500 name="left_upper_arm_motor1" rpy="${radians(180)} ${radians(180)} ${radians(-90)}"/>
+        <xacro:upper_arm name="left_upper_arm"/>
+        <xacro:dynamixel_pro_h54-100-s500 name="left_upper_arm_motor2" rpy="0 ${radians(90)} ${radians(90)}"/>
+        <joint name="left_upper_arm_joint" type="continuous">
+            <origin xyz="0.045 -0.0505 0" rpy="${radians(-90)} 0 0"/>
+            <parent link="left_shoulder"/>
+            <child link="left_upper_arm_motor1"/>
+            <axis xyz="1 0 0"/>
+        </joint>
+        <joint name="left_upper_arm_internal_mount1" type="fixed">
+            <origin xyz="0.00005 0 0" rpy="0 0 0"/>
+            <parent link="left_upper_arm_motor1"/>
+            <child link="left_upper_arm"/>
+        </joint>
+        <joint name="left_upper_arm_internal_mount2" type="fixed">
+            <origin xyz="0.01495 -0.25 0" rpy="0 0 0"/>
+            <parent link="left_upper_arm"/>
+            <child link="left_upper_arm_motor2"/>
         </joint>
     </xacro:macro>
@@ -70,4 +117,20 @@
         </joint>
     </xacro:macro>
+    <!-- left_lower_arm -->
+    <xacro:macro name="left_lower_arm">
+        <xacro:lower_arm name="left_lower_arm"/>
+        <xacro:dynamixel_pro_h42-20-s300 name="left_lower_arm_motor" rpy="0 0 ${radians(-90)}"/>
+        <joint name="left_lower_arm_joint" type="continuous">
+            <origin xyz="0 0 0" rpy="0 0 0"/>
+            <parent link="left_upper_arm_motor2"/>
+            <child link="left_lower_arm"/>
+            <axis xyz="1 0 0"/>
+        </joint>
+        <joint name="left_lower_arm_internal_mount" type="fixed">
+            <origin xyz="0.0405 -0.2 0" rpy="0 0 0"/>
+            <parent link="left_lower_arm"/>
+            <child link="left_lower_arm_motor"/>
+        </joint>
+    </xacro:macro>
     <!-- right_wrist -->
     <xacro:macro name="right_wrist">
@@ -75,5 +138,5 @@
         <xacro:dynamixel_pro_h42-20-s300 name="right_wrist_motor" rpy="0 ${radians(-90)} ${radians(180)}"/>
         <joint name="right_wrist_joint" type="continuous">
-            <origin xyz="0 0 0" rpy="0 0 0"/>
+            <origin xyz="0 0 0" rpy="${radians(90)} 0 0"/>
             <parent link="right_lower_arm_motor"/>
             <child link="right_wrist"/>
@@ -84,4 +147,20 @@
             <parent link="right_wrist"/>
             <child link="right_wrist_motor"/>
+        </joint>
+    </xacro:macro>
+    <!-- left_wrist -->
+    <xacro:macro name="left_wrist">
+        <xacro:wrist name="left_wrist"/>
+        <xacro:dynamixel_pro_h42-20-s300 name="left_wrist_motor" rpy="0 ${radians(-90)} ${radians(180)}"/>
+        <joint name="left_wrist_joint" type="continuous">
+            <origin xyz="0 0 0" rpy="${radians(-90)} 0 0"/>
+            <parent link="left_lower_arm_motor"/>
+            <child link="left_wrist"/>
+            <axis xyz="1 0 0"/>
+        </joint>
+        <joint name="left_wrist_internal_mount" type="fixed">
+            <origin xyz="0.035 -0.055 0" rpy="0 0 0"/>
+            <parent link="left_wrist"/>
+            <child link="left_wrist_motor"/>
         </joint>
     </xacro:macro>
@@ -102,3 +181,19 @@
         </joint>
     </xacro:macro>
+    <!-- left_palm -->
+    <xacro:macro name="left_palm">
+        <xacro:wrist name="left_palm"/>
+        <xacro:dynamixel_pro_h42-20-s300 name="left_palm_motor" rpy="0 ${radians(-90)} ${radians(180)}"/>
+        <joint name="left_palm_joint" type="continuous">
+            <origin xyz="0 0 0" rpy="0 ${radians(180)} ${radians(90)}"/>
+            <parent link="left_wrist_motor"/>
+            <child link="left_palm"/>
+            <axis xyz="1 0 0"/>
+        </joint>
+        <joint name="left_palm_internal_mount" type="fixed">
+            <origin xyz="0.035 -0.055 0" rpy="0 0 0"/>
+            <parent link="left_palm"/>
+            <child link="left_palm_motor"/>
+        </joint>
+    </xacro:macro>
 </robot>
