Commit message: added covers

File: urdf/parts.xacro (robot description, xacro)
@@ -5,4 +5,6 @@
     <xacro:property name="triple_zero" value="0 0 0"/>
     <xacro:property name="link_material" value="Light_grey"/>
+    <xacro:property name="cover_material" value="Black"/>
+    <xacro:property name="extension_ring_material" value="White"/>
     <xacro:property name="motor_material" value="Grey"/>
     <!-- links -->
@@ -157,4 +159,185 @@
         </gazebo>
     </xacro:macro>
+    <!-- covers -->
+    <!-- shoulder_extension_ring -->
+    <xacro:macro name="shoulder_extension_ring" params="name xyz:=${triple_zero} rpy:=${triple_zero}">
+        <link name="${name}">
+            <inertial>
+                <origin xyz="${xyz}" rpy="${rpy}"/>
+                <mass value="0.01"/>
+                <inertia
+                    ixx="0.000008154" ixy="0" ixz="0"
+                    iyy="0.000007974" iyz="0.000000006"
+                    izz="0.000015238"
+                />
+            </inertial>
+            <visual>
+                <origin xyz="${xyz}" rpy="${rpy}"/>
+                <geometry>
+                    <mesh filename="package://separable_jaws_description/meshes/shoulder_extension_ring.stl"/>
+                </geometry>
+                <material name="${extension_ring_material}"/>
+            </visual>
+            <collision>
+                <origin xyz="${xyz}" rpy="${rpy}"/>
+                <geometry>
+                    <mesh filename="package://separable_jaws_description/meshes/shoulder_extension_ring.stl"/>
+                </geometry>
+            </collision>
+        </link>
+        <gazebo reference="${name}">
+            <material>Gazebo/${extension_ring_material}</material>
+        </gazebo>
+    </xacro:macro>
+    <!-- shoulder_cover -->
+    <xacro:macro name="shoulder_cover" params="name xyz:=${triple_zero} rpy:=${triple_zero}">
+        <link name="${name}">
+            <inertial>
+                <origin xyz="${xyz}" rpy="${rpy}"/>
+                <mass value="0.075"/>
+                <inertia
+                    ixx="0.000055846" ixy="0" ixz="0"
+                    iyy="0.000055846" iyz="0"
+                    izz="0.000068514"
+                />
+            </inertial>
+            <visual>
+                <origin xyz="${xyz}" rpy="${rpy}"/>
+                <geometry>
+                    <mesh filename="package://separable_jaws_description/meshes/shoulder_cover.stl"/>
+                </geometry>
+                <material name="${cover_material}"/>
+            </visual>
+            <collision>
+                <origin xyz="${xyz}" rpy="${rpy}"/>
+                <geometry>
+                    <mesh filename="package://separable_jaws_description/meshes/shoulder_cover.stl"/>
+                </geometry>
+            </collision>
+        </link>
+        <gazebo reference="${name}">
+            <material>Gazebo/${cover_material}</material>
+        </gazebo>
+    </xacro:macro>
+    <!-- upper_arm_cover -->
+    <xacro:macro name="upper_arm_cover" params="name xyz:=${triple_zero} rpy:=${triple_zero}">
+        <link name="${name}">
+            <inertial>
+                <origin xyz="${xyz}" rpy="${rpy}"/>
+                <mass value="0.235"/>
+                <inertia
+                    ixx="0.000385567" ixy="-0.00000002" ixz="0.000732197"
+                    iyy="0.006196229" iyz="-0.000000009"
+                    izz="0.00621496"
+                />
+            </inertial>
+            <visual>
+                <origin xyz="${xyz}" rpy="${rpy}"/>
+                <geometry>
+                    <mesh filename="package://separable_jaws_description/meshes/upper_arm_cover.stl"/>
+                </geometry>
+                <material name="${cover_material}"/>
+            </visual>
+            <collision>
+                <origin xyz="${xyz}" rpy="${rpy}"/>
+                <geometry>
+                    <mesh filename="package://separable_jaws_description/meshes/upper_arm_cover.stl"/>
+                </geometry>
+            </collision>
+        </link>
+        <gazebo reference="${name}">
+            <material>Gazebo/${cover_material}</material>
+        </gazebo>
+    </xacro:macro>
+    <!-- lower_arm_cover -->
+    <xacro:macro name="lower_arm_cover" params="name xyz:=${triple_zero} rpy:=${triple_zero}">
+        <link name="${name}">
+            <inertial>
+                <origin xyz="${xyz}" rpy="${rpy}"/>
+                <mass value="0.079"/>
+                <inertia
+                    ixx="0.000047626" ixy="0.000000367" ixz="0.000039299"
+                    iyy="0.001178645" iyz="-0.000000021"
+                    izz="0.00121964"
+                />
+            </inertial>
+            <visual>
+                <origin xyz="${xyz}" rpy="${rpy}"/>
+                <geometry>
+                    <mesh filename="package://separable_jaws_description/meshes/lower_arm_cover.stl"/>
+                </geometry>
+                <material name="${cover_material}"/>
+            </visual>
+            <collision>
+                <origin xyz="${xyz}" rpy="${rpy}"/>
+                <geometry>
+                    <mesh filename="package://separable_jaws_description/meshes/lower_arm_cover.stl"/>
+                </geometry>
+            </collision>
+        </link>
+        <gazebo reference="${name}">
+            <material>Gazebo/${cover_material}</material>
+        </gazebo>
+    </xacro:macro>
+    <!-- wrist_extension_ring -->
+    <xacro:macro name="wrist_extension_ring" params="name xyz:=${triple_zero} rpy:=${triple_zero}">
+        <link name="${name}">
+            <inertial>
+                <origin xyz="${xyz}" rpy="${rpy}"/>
+                <mass value="0.007"/>
+                <inertia
+                    ixx="0.000003276" ixy="0" ixz="0"
+                    iyy="0.000003197" iyz="0.000000003"
+                    izz="0.00000617"
+                />
+            </inertial>
+            <visual>
+                <origin xyz="${xyz}" rpy="${rpy}"/>
+                <geometry>
+                    <mesh filename="package://separable_jaws_description/meshes/wrist_extension_ring.stl"/>
+                </geometry>
+                <material name="${extension_ring_material}"/>
+            </visual>
+            <collision>
+                <origin xyz="${xyz}" rpy="${rpy}"/>
+                <geometry>
+                    <mesh filename="package://separable_jaws_description/meshes/wrist_extension_ring.stl"/>
+                </geometry>
+            </collision>
+        </link>
+        <gazebo reference="${name}">
+            <material>Gazebo/${extension_ring_material}</material>
+        </gazebo>
+    </xacro:macro>
+    <!-- wrist_cover -->
+    <xacro:macro name="wrist_cover" params="name xyz:=${triple_zero} rpy:=${triple_zero}">
+        <link name="${name}">
+            <inertial>
+                <origin xyz="${xyz}" rpy="${rpy}"/>
+                <mass value="0.037"/>
+                <inertia
+                    ixx="0.000009686" ixy="0" ixz="0"
+                    iyy="0.00000987" iyz="0"
+                    izz="0.000017485"
+                />
+            </inertial>
+            <visual>
+                <origin xyz="${xyz}" rpy="${rpy}"/>
+                <geometry>
+                    <mesh filename="package://separable_jaws_description/meshes/wrist_cover.stl"/>
+                </geometry>
+                <material name="${cover_material}"/>
+            </visual>
+            <collision>
+                <origin xyz="${xyz}" rpy="${rpy}"/>
+                <geometry>
+                    <mesh filename="package://separable_jaws_description/meshes/wrist_cover.stl"/>
+                </geometry>
+            </collision>
+        </link>
+        <gazebo reference="${name}">
+            <material>Gazebo/${cover_material}</material>
+        </gazebo>
+    </xacro:macro>
     <!-- motors -->
     <!-- dynamixel_pro_h54-100-s500 -->

File: urdf/subassemblies.xacro (robot description, xacro)
@@ -29,4 +29,6 @@
         <xacro:dynamixel_pro_h54-100-s500 name="right_shoulder_motor" rpy="0 ${radians(90)} 0"/>
         <xacro:shoulder name="right_shoulder"/>
+        <xacro:shoulder_extension_ring name="right_shoulder_extension_ring"/>
+        <xacro:shoulder_cover name="right_shoulder_cover"/>
         <joint name="right_shoulder_joint" type="continuous">
             <origin xyz="0 -0.025 0" rpy="0 0 0"/>
@@ -35,8 +37,18 @@
             <axis xyz="0 -1 0"/>
         </joint>
-        <joint name="right_shoulder_internal_mount" type="fixed">
+        <joint name="right_shoulder_internal_mount1" type="fixed">
             <origin xyz="0 -0.00005 0" rpy="0 ${radians(-90)} 0"/>
             <parent link="right_shoulder_motor"/>
             <child link="right_shoulder"/>
+        </joint>
+        <joint name="right_shoulder_internal_mount2" type="fixed">
+            <origin xyz="0 -0.1 0" rpy="${radians(90)} ${radians(-90)} 0"/>
+            <parent link="right_shoulder"/>
+            <child link="right_shoulder_extension_ring"/>
+        </joint>
+        <joint name="right_shoulder_internal_mount3" type="fixed">
+            <origin xyz="0 0 0.012" rpy="0 0 0"/>
+            <parent link="right_shoulder_extension_ring"/>
+            <child link="right_shoulder_cover"/>
         </joint>
     </xacro:macro>
@@ -45,4 +57,6 @@
         <xacro:dynamixel_pro_h54-100-s500 name="left_shoulder_motor" rpy="0 ${radians(-90)} 0"/>
         <xacro:shoulder name="left_shoulder"/>
+        <xacro:shoulder_extension_ring name="left_shoulder_extension_ring"/>
+        <xacro:shoulder_cover name="left_shoulder_cover"/>
         <joint name="left_shoulder_joint" type="continuous">
             <origin xyz="0 -0.025 0" rpy="0 ${radians(180)} 0"/>
@@ -51,8 +65,18 @@
             <axis xyz="0 -1 0"/>
         </joint>
-        <joint name="left_shoulder_internal_mount" type="fixed">
+        <joint name="left_shoulder_internal_mount1" type="fixed">
             <origin xyz="0 -0.00005 0" rpy="0 ${radians(-90)} 0"/>
             <parent link="left_shoulder_motor"/>
             <child link="left_shoulder"/>
+        </joint>
+        <joint name="left_shoulder_internal_mount2" type="fixed">
+            <origin xyz="0 -0.1 0" rpy="${radians(90)} ${radians(-90)} 0"/>
+            <parent link="left_shoulder"/>
+            <child link="left_shoulder_extension_ring"/>
+        </joint>
+        <joint name="left_shoulder_internal_mount3" type="fixed">
+            <origin xyz="0 0 0.012" rpy="0 0 0"/>
+            <parent link="left_shoulder_extension_ring"/>
+            <child link="left_shoulder_cover"/>
         </joint>
     </xacro:macro>
@@ -61,4 +85,5 @@
         <xacro:dynamixel_pro_h54-200-s500 name="right_upper_arm_motor1" rpy="${radians(180)} 0 ${radians(-90)}"/>
         <xacro:upper_arm name="right_upper_arm"/>
+        <xacro:upper_arm_cover name="right_upper_arm_cover"/>
         <xacro:dynamixel_pro_h54-100-s500 name="right_upper_arm_motor2" rpy="0 ${radians(90)} ${radians(90)}"/>
         <joint name="right_upper_arm_joint" type="continuous">
@@ -78,4 +103,9 @@
             <child link="right_upper_arm_motor2"/>
         </joint>
+        <joint name="right_upper_arm_internal_mount3" type="fixed">
+            <origin xyz="0.1 0 0" rpy="${radians(90)} 0 ${radians(-90)}"/>
+            <parent link="right_upper_arm"/>
+            <child link="right_upper_arm_cover"/>
+        </joint>
     </xacro:macro>
     <!-- left_upper_arm -->
@@ -83,4 +113,5 @@
         <xacro:dynamixel_pro_h54-200-s500 name="left_upper_arm_motor1" rpy="${radians(180)} ${radians(180)} ${radians(-90)}"/>
         <xacro:upper_arm name="left_upper_arm"/>
+        <xacro:upper_arm_cover name="left_upper_arm_cover"/>
         <xacro:dynamixel_pro_h54-100-s500 name="left_upper_arm_motor2" rpy="0 ${radians(90)} ${radians(90)}"/>
         <joint name="left_upper_arm_joint" type="continuous">
@@ -100,8 +131,14 @@
             <child link="left_upper_arm_motor2"/>
         </joint>
+        <joint name="left_upper_arm_internal_mount3" type="fixed">
+            <origin xyz="0.1 0 0" rpy="${radians(90)} 0 ${radians(-90)}"/>
+            <parent link="left_upper_arm"/>
+            <child link="left_upper_arm_cover"/>
+        </joint>
     </xacro:macro>
     <!-- right_lower_arm -->
     <xacro:macro name="right_lower_arm">
         <xacro:lower_arm name="right_lower_arm"/>
+        <xacro:lower_arm_cover name="right_lower_arm_cover"/>
         <xacro:dynamixel_pro_h42-20-s300 name="right_lower_arm_motor" rpy="0 ${radians(180)} ${radians(-90)}"/>
         <joint name="right_lower_arm_joint" type="continuous">
@@ -111,13 +148,19 @@
             <axis xyz="1 0 0"/>
         </joint>
-        <joint name="right_lower_arm_internal_mount" type="fixed">
+        <joint name="right_lower_arm_internal_mount1" type="fixed">
             <origin xyz="0.0405 -0.2 0" rpy="0 0 0"/>
             <parent link="right_lower_arm"/>
             <child link="right_lower_arm_motor"/>
         </joint>
+        <joint name="right_lower_arm_internal_mount2" type="fixed">
+            <origin xyz="-0.05 0 0" rpy="${radians(-90)} 0 ${radians(90)}"/>
+            <parent link="right_lower_arm"/>
+            <child link="right_lower_arm_cover"/>
+        </joint>
     </xacro:macro>
     <!-- left_lower_arm -->
     <xacro:macro name="left_lower_arm">
         <xacro:lower_arm name="left_lower_arm"/>
+        <xacro:lower_arm_cover name="left_lower_arm_cover"/>
         <xacro:dynamixel_pro_h42-20-s300 name="left_lower_arm_motor" rpy="0 0 ${radians(-90)}"/>
         <joint name="left_lower_arm_joint" type="continuous">
@@ -132,8 +175,15 @@
             <child link="left_lower_arm_motor"/>
         </joint>
+        <joint name="left_lower_arm_internal_mount2" type="fixed">
+            <origin xyz="-0.05 0 0" rpy="${radians(-90)} 0 ${radians(90)}"/>
+            <parent link="left_lower_arm"/>
+            <child link="left_lower_arm_cover"/>
+        </joint>
     </xacro:macro>
     <!-- right_wrist -->
     <xacro:macro name="right_wrist">
         <xacro:wrist name="right_wrist"/>
+        <xacro:wrist_extension_ring name="right_wrist_extension_ring"/>
+        <xacro:wrist_cover name="right_wrist_cover"/>
         <xacro:dynamixel_pro_h42-20-s300 name="right_wrist_motor" rpy="0 ${radians(-90)} ${radians(180)}"/>
         <joint name="right_wrist_joint" type="continuous">
@@ -143,8 +193,18 @@
             <axis xyz="1 0 0"/>
         </joint>
-        <joint name="right_wrist_internal_mount" type="fixed">
+        <joint name="right_wrist_internal_mount1" type="fixed">
             <origin xyz="0.035 -0.055 0" rpy="0 0 0"/>
             <parent link="right_wrist"/>
             <child link="right_wrist_motor"/>
+        </joint>
+        <joint name="right_wrist_internal_mount2" type="fixed">
+            <origin xyz="0.035 0.035 0" rpy="${radians(-90)} ${radians(-90)} 0"/>
+            <parent link="right_wrist"/>
+            <child link="right_wrist_extension_ring"/>
+        </joint>
+        <joint name="right_wrist_internal_mount3" type="fixed">
+            <origin xyz="0 0 0.009" rpy="0 0 0"/>
+            <parent link="right_wrist_extension_ring"/>
+            <child link="right_wrist_cover"/>
         </joint>
     </xacro:macro>
@@ -152,4 +212,6 @@
     <xacro:macro name="left_wrist">
         <xacro:wrist name="left_wrist"/>
+        <xacro:wrist_extension_ring name="left_wrist_extension_ring"/>
+        <xacro:wrist_cover name="left_wrist_cover"/>
         <xacro:dynamixel_pro_h42-20-s300 name="left_wrist_motor" rpy="0 ${radians(-90)} ${radians(180)}"/>
         <joint name="left_wrist_joint" type="continuous">
@@ -159,8 +221,18 @@
             <axis xyz="1 0 0"/>
         </joint>
-        <joint name="left_wrist_internal_mount" type="fixed">
+        <joint name="left_wrist_internal_mount1" type="fixed">
             <origin xyz="0.035 -0.055 0" rpy="0 0 0"/>
             <parent link="left_wrist"/>
             <child link="left_wrist_motor"/>
+        </joint>
+        <joint name="left_wrist_internal_mount2" type="fixed">
+            <origin xyz="0.035 0.035 0" rpy="${radians(-90)} ${radians(-90)} 0"/>
+            <parent link="left_wrist"/>
+            <child link="left_wrist_extension_ring"/>
+        </joint>
+        <joint name="left_wrist_internal_mount3" type="fixed">
+            <origin xyz="0 0 0.009" rpy="0 0 0"/>
+            <parent link="left_wrist_extension_ring"/>
+            <child link="left_wrist_cover"/>
         </joint>
     </xacro:macro>
@@ -168,4 +240,6 @@
     <xacro:macro name="right_palm">
         <xacro:wrist name="right_palm"/>
+        <xacro:wrist_extension_ring name="right_palm_extension_ring"/>
+        <xacro:wrist_cover name="right_palm_cover"/>
         <xacro:dynamixel_pro_h42-20-s300 name="right_palm_motor" rpy="0 ${radians(-90)} ${radians(180)}"/>
         <joint name="right_palm_joint" type="continuous">
@@ -175,8 +249,18 @@
             <axis xyz="1 0 0"/>
         </joint>
-        <joint name="right_palm_internal_mount" type="fixed">
+        <joint name="right_palm_internal_mount1" type="fixed">
             <origin xyz="0.035 -0.055 0" rpy="0 0 0"/>
             <parent link="right_palm"/>
             <child link="right_palm_motor"/>
+        </joint>
+        <joint name="right_palm_internal_mount2" type="fixed">
+            <origin xyz="0.035 0.035 0" rpy="${radians(-90)} ${radians(-90)} 0"/>
+            <parent link="right_palm"/>
+            <child link="right_palm_extension_ring"/>
+        </joint>
+        <joint name="right_palm_internal_mount3" type="fixed">
+            <origin xyz="0 0 0.009" rpy="0 0 0"/>
+            <parent link="right_palm_extension_ring"/>
+            <child link="right_palm_cover"/>
         </joint>
     </xacro:macro>
@@ -184,4 +268,6 @@
     <xacro:macro name="left_palm">
         <xacro:wrist name="left_palm"/>
+        <xacro:wrist_extension_ring name="left_palm_extension_ring"/>
+        <xacro:wrist_cover name="left_palm_cover"/>
         <xacro:dynamixel_pro_h42-20-s300 name="left_palm_motor" rpy="0 ${radians(-90)} ${radians(180)}"/>
         <joint name="left_palm_joint" type="continuous">
@@ -191,9 +277,19 @@
             <axis xyz="1 0 0"/>
         </joint>
-        <joint name="left_palm_internal_mount" type="fixed">
+        <joint name="left_palm_internal_mount1" type="fixed">
             <origin xyz="0.035 -0.055 0" rpy="0 0 0"/>
             <parent link="left_palm"/>
             <child link="left_palm_motor"/>
         </joint>
+        <joint name="left_palm_internal_mount2" type="fixed">
+            <origin xyz="0.035 0.035 0" rpy="${radians(-90)} ${radians(-90)} 0"/>
+            <parent link="left_palm"/>
+            <child link="left_palm_extension_ring"/>
+        </joint>
+        <joint name="left_palm_internal_mount3" type="fixed">
+            <origin xyz="0 0 0.009" rpy="0 0 0"/>
+            <parent link="left_palm_extension_ring"/>
+            <child link="left_palm_cover"/>
+        </joint>
     </xacro:macro>
 </robot>
