Commit message: add joint limit

File: urdf/parts.xacro (robot description, xacro)
@@ -35,7 +35,9 @@
             </collision>
         </link>
-        <gazebo reference="${name}">
-            <material>Gazebo/${link_material}</material>
-        </gazebo>
+        <xacro:if value="$(arg using_gazebo)">
+            <gazebo reference="${name}">
+                <material>Gazebo/${link_material}</material>
+            </gazebo>
+        </xacro:if>
     </xacro:macro>
     <!-- shoulder -->
@@ -65,7 +67,9 @@
             </collision>
         </link>
-        <gazebo reference="${name}">
-            <material>Gazebo/${link_material}</material>
-        </gazebo>
+        <xacro:if value="$(arg using_gazebo)">
+            <gazebo reference="${name}">
+                <material>Gazebo/${link_material}</material>
+            </gazebo>
+        </xacro:if>
     </xacro:macro>
     <!-- upper_arm -->
@@ -95,7 +99,9 @@
             </collision>
         </link>
-        <gazebo reference="${name}">
-            <material>Gazebo/${link_material}</material>
-        </gazebo>
+        <xacro:if value="$(arg using_gazebo)">
+            <gazebo reference="${name}">
+                <material>Gazebo/${link_material}</material>
+            </gazebo>
+        </xacro:if>
     </xacro:macro>
     <!-- lower_arm -->
@@ -125,7 +131,9 @@
             </collision>
         </link>
-        <gazebo reference="${name}">
-            <material>Gazebo/${link_material}</material>
-        </gazebo>
+        <xacro:if value="$(arg using_gazebo)">
+            <gazebo reference="${name}">
+                <material>Gazebo/${link_material}</material>
+            </gazebo>
+        </xacro:if>
     </xacro:macro>
     <!-- wrist -->
@@ -155,7 +163,9 @@
             </collision>
         </link>
-        <gazebo reference="${name}">
-            <material>Gazebo/${link_material}</material>
-        </gazebo>
+        <xacro:if value="$(arg using_gazebo)">
+            <gazebo reference="${name}">
+                <material>Gazebo/${link_material}</material>
+            </gazebo>
+        </xacro:if>
     </xacro:macro>
     <!-- covers -->
@@ -186,7 +196,9 @@
             </collision>
         </link>
-        <gazebo reference="${name}">
-            <material>Gazebo/${extension_ring_material}</material>
-        </gazebo>
+        <xacro:if value="$(arg using_gazebo)">
+            <gazebo reference="${name}">
+                <material>Gazebo/${extension_ring_material}</material>
+            </gazebo>
+        </xacro:if>
     </xacro:macro>
     <!-- shoulder_cover -->
@@ -216,7 +228,9 @@
             </collision>
         </link>
-        <gazebo reference="${name}">
-            <material>Gazebo/${cover_material}</material>
-        </gazebo>
+        <xacro:if value="$(arg using_gazebo)">
+            <gazebo reference="${name}">
+                <material>Gazebo/${cover_material}</material>
+            </gazebo>
+        </xacro:if>
     </xacro:macro>
     <!-- upper_arm_cover -->
@@ -246,7 +260,9 @@
             </collision>
         </link>
-        <gazebo reference="${name}">
-            <material>Gazebo/${cover_material}</material>
-        </gazebo>
+        <xacro:if value="$(arg using_gazebo)">
+            <gazebo reference="${name}">
+                <material>Gazebo/${cover_material}</material>
+            </gazebo>
+        </xacro:if>
     </xacro:macro>
     <!-- lower_arm_cover -->
@@ -276,7 +292,9 @@
             </collision>
         </link>
-        <gazebo reference="${name}">
-            <material>Gazebo/${cover_material}</material>
-        </gazebo>
+        <xacro:if value="$(arg using_gazebo)">
+            <gazebo reference="${name}">
+                <material>Gazebo/${cover_material}</material>
+            </gazebo>
+        </xacro:if>
     </xacro:macro>
     <!-- wrist_extension_ring -->
@@ -306,7 +324,9 @@
             </collision>
         </link>
-        <gazebo reference="${name}">
-            <material>Gazebo/${extension_ring_material}</material>
-        </gazebo>
+        <xacro:if value="$(arg using_gazebo)">
+            <gazebo reference="${name}">
+                <material>Gazebo/${extension_ring_material}</material>
+            </gazebo>
+        </xacro:if>
     </xacro:macro>
     <!-- wrist_cover -->
@@ -336,7 +356,9 @@
             </collision>
         </link>
-        <gazebo reference="${name}">
-            <material>Gazebo/${cover_material}</material>
-        </gazebo>
+        <xacro:if value="$(arg using_gazebo)">
+            <gazebo reference="${name}">
+                <material>Gazebo/${cover_material}</material>
+            </gazebo>
+        </xacro:if>
     </xacro:macro>
     <!-- motors -->
@@ -367,7 +389,9 @@
             </collision>
         </link>
-        <gazebo reference="${name}">
-            <material>Gazebo/${motor_material}</material>
-        </gazebo>
+        <xacro:if value="$(arg using_gazebo)">
+            <gazebo reference="${name}">
+                <material>Gazebo/${motor_material}</material>
+            </gazebo>
+        </xacro:if>
     </xacro:macro>
     <!-- dynamixel_pro_h54-200-s500 -->
@@ -397,7 +421,9 @@
             </collision>
         </link>
-        <gazebo reference="${name}">
-            <material>Gazebo/${motor_material}</material>
-        </gazebo>
+        <xacro:if value="$(arg using_gazebo)">
+            <gazebo reference="${name}">
+                <material>Gazebo/${motor_material}</material>
+            </gazebo>
+        </xacro:if>
     </xacro:macro>
     <!-- dynamixel_pro_h42-20-s300-->
@@ -427,7 +453,9 @@
             </collision>
         </link>
-        <gazebo reference="${name}">
-            <material>Gazebo/${motor_material}</material>
-        </gazebo>
+        <xacro:if value="$(arg using_gazebo)">
+            <gazebo reference="${name}">
+                <material>Gazebo/${motor_material}</material>
+            </gazebo>
+        </xacro:if>
     </xacro:macro>
 </robot>

File: urdf/ros2_control.xacro (robot description, xacro)
@@ -2,8 +2,7 @@
 <robot name="separable_jaws" xmlns:xacro="http://www.ros.org/wiki/xacro">
     <!-- joint control config macro -->
-    <xacro:macro name="joint_control_config" params="joint_name id:=0 model pos_max:=${radians(180)} pos_min:=${radians(-180)}">
+    <xacro:macro name="joint_control_config" params="joint_name id:=0 pos_max:=${radians(180)} pos_min:=${radians(-180)}">
         <joint name="${joint_name}">
             <param name="id">${id}</param>
-            <param name="model">${model}</param>
             <command_interface name="position">
                 <param name="min">${pos_max}</param>
@@ -11,6 +10,4 @@
             </command_interface>
             <command_interface name="velocity"/>
-            <command_interface name="acceleration"/>
-            <command_interface name="effort"/>
             <state_interface name="position"/>
             <state_interface name="velocity"/>
@@ -22,20 +19,32 @@
         <ros2_control name="separable_jaws_control_system" type="system">
             <hardware>
-                <plugin>dynamixel_controller/DynamixelHardwareInterface</plugin>
-                <param name="dynamixel_port">/dev/ttyUSB0</param>
-                <param name="dynamixel_protocol">2.0</param>
-                <param name="dynamixel_baudrate">1000000</param>
-                <param name="dynamixel_control_table">$(find dynamixel_controller)/doc/dynamixel_control_table.yaml</param>
+                <xacro:if value="$(arg using_gazebo)">
+                    <plugin>gazebo_ros2_control/GazeboSystem</plugin>
+                </xacro:if>
+                <xacro:unless value="$(arg using_gazebo)">
+                    <xacro:if value="$(arg using_fake_hardware)">
+                        <plugin>mock_components/GenericSystem</plugin>
+                    </xacro:if>
+                    <xacro:unless value="$(arg using_fake_hardware)">
+                        <plugin>dynamixel_hardware/DynamixelHardware</plugin>
+                        <param name="usb_port">/dev/ttyUSB0</param>
+                        <param name="baud_rate">1000000</param>
+                    </xacro:unless>
+                </xacro:unless>
             </hardware>
-            <xacro:joint_control_config joint_name="right_shoulder_joint" id="1" model="H54_100_S500_R"/>
-            <xacro:joint_control_config joint_name="right_upper_arm_joint" id="2" model="H54_200_S500_R"/>
-            <xacro:joint_control_config joint_name="right_lower_arm_joint" id="3" model="H54_100_S500_R"/>
-            <xacro:joint_control_config joint_name="right_wrist_joint" id="4" model="H42_20_S300_R"/>
-            <xacro:joint_control_config joint_name="right_palm_joint" id="5" model="H42_20_S300_R"/>
-            <xacro:joint_control_config joint_name="left_shoulder_joint" id="7" model="H54_100_S500_R"/>
-            <xacro:joint_control_config joint_name="left_upper_arm_joint" id="8" model="H54_200_S500_R"/>
-            <xacro:joint_control_config joint_name="left_lower_arm_joint" id="9" model="H54_100_S500_R"/>
-            <xacro:joint_control_config joint_name="left_wrist_joint" id="10" model="H42_20_S300_R"/>
-            <xacro:joint_control_config joint_name="left_palm_joint" id="11" model="H42_20_S300_R"/>
+            <xacro:if value="$(arg using_left_arm)">
+                <xacro:joint_control_config joint_name="left_shoulder_joint" id="7"/>
+                <xacro:joint_control_config joint_name="left_upper_arm_joint" id="8"/>
+                <xacro:joint_control_config joint_name="left_lower_arm_joint" id="9"/>
+                <xacro:joint_control_config joint_name="left_wrist_joint" id="10"/>
+                <xacro:joint_control_config joint_name="left_palm_joint" id="11"/>
+            </xacro:if>
+            <xacro:if value="$(arg using_right_arm)">
+                <xacro:joint_control_config joint_name="right_shoulder_joint" id="1"/>
+                <xacro:joint_control_config joint_name="right_upper_arm_joint" id="2"/>
+                <xacro:joint_control_config joint_name="right_lower_arm_joint" id="3"/>
+                <xacro:joint_control_config joint_name="right_wrist_joint" id="4"/>
+                <xacro:joint_control_config joint_name="right_palm_joint" id="5"/>
+            </xacro:if>
         </ros2_control>
     </xacro:macro>

File: urdf/separable_jaws.xacro (robot description, xacro)
@@ -1,4 +1,9 @@
 <?xml version="1.0"?>
 <robot name="separable_jaws" xmlns:xacro="http://www.ros.org/wiki/xacro">
+    <!-- declare arguments -->
+    <xacro:arg name="using_left_arm" default="true"/>
+    <xacro:arg name="using_right_arm" default="true"/>
+    <xacro:arg name="using_gazebo" default="false"/>
+    <xacro:arg name="using_fake_hardware" default="true"/>
     <!-- include macros from other files-->
     <xacro:include filename="$(find separable_jaws_description)/urdf/material.xacro"/>
@@ -8,16 +13,20 @@
     <!-- robot definition -->
     <link name="base_link"/>
-    <xacro:right_bracket xyz="0 -0.05 0"/>
-    <xacro:right_shoulder/>
-    <xacro:right_upper_arm/>
-    <xacro:right_lower_arm/>
-    <xacro:right_wrist/>
-    <xacro:right_palm/>
-    <xacro:left_bracket xyz="0 0.05 0"/>
-    <xacro:left_shoulder/>
-    <xacro:left_upper_arm/>
-    <xacro:left_lower_arm/>
-    <xacro:left_wrist/>
-    <xacro:left_palm/>
+    <xacro:if value="$(arg using_left_arm)">
+        <xacro:left_bracket xyz="0 0.05 0.2"/>
+        <xacro:left_shoulder/>
+        <xacro:left_upper_arm/>
+        <xacro:left_lower_arm/>
+        <xacro:left_wrist/>
+        <xacro:left_palm/>
+    </xacro:if>
+    <xacro:if value="$(arg using_right_arm)">
+        <xacro:right_bracket xyz="0 -0.05 0.2"/>
+        <xacro:right_shoulder/>
+        <xacro:right_upper_arm/>
+        <xacro:right_lower_arm/>
+        <xacro:right_wrist/>
+        <xacro:right_palm/>
+    </xacro:if>
     <xacro:separable_jaws_ros2_control/>
 </robot>
