Commit message: refresh the urdf file and add rviz config

File: urdf/parts.xacro (robot description, xacro)
@@ -5,4 +5,6 @@
     <xacro:property name="triple_zero" value="0 0 0"/>
     <xacro:property name="link_material" value="Light_grey"/>
+    <xacro:property name="cover_material" value="Black"/>
+    <xacro:property name="extension_ring_material" value="White"/>
     <xacro:property name="motor_material" value="Grey"/>
     <!-- links -->
@@ -33,7 +35,9 @@
             </collision>
         </link>
-        <gazebo reference="${name}">
-            <material>Gazebo/${link_material}</material>
-        </gazebo>
+        <xacro:if value="$(arg using_gazebo)">
+            <gazebo reference="${name}">
+                <material>Gazebo/${link_material}</material>
+            </gazebo>
+        </xacro:if>
     </xacro:macro>
     <!-- shoulder -->
@@ -63,7 +67,9 @@
             </collision>
         </link>
-        <gazebo reference="${name}">
-            <material>Gazebo/${link_material}</material>
-        </gazebo>
+        <xacro:if value="$(arg using_gazebo)">
+            <gazebo reference="${name}">
+                <material>Gazebo/${link_material}</material>
+            </gazebo>
+        </xacro:if>
     </xacro:macro>
     <!-- upper_arm -->
@@ -93,7 +99,9 @@
             </collision>
         </link>
-        <gazebo reference="${name}">
-            <material>Gazebo/${link_material}</material>
-        </gazebo>
+        <xacro:if value="$(arg using_gazebo)">
+            <gazebo reference="${name}">
+                <material>Gazebo/${link_material}</material>
+            </gazebo>
+        </xacro:if>
     </xacro:macro>
     <!-- lower_arm -->
@@ -123,7 +131,9 @@
             </collision>
         </link>
-        <gazebo reference="${name}">
-            <material>Gazebo/${link_material}</material>
-        </gazebo>
+        <xacro:if value="$(arg using_gazebo)">
+            <gazebo reference="${name}">
+                <material>Gazebo/${link_material}</material>
+            </gazebo>
+        </xacro:if>
     </xacro:macro>
     <!-- wrist -->
@@ -153,7 +163,202 @@
             </collision>
         </link>
-        <gazebo reference="${name}">
-            <material>Gazebo/${link_material}</material>
-        </gazebo>
+        <xacro:if value="$(arg using_gazebo)">
+            <gazebo reference="${name}">
+                <material>Gazebo/${link_material}</material>
+            </gazebo>
+        </xacro:if>
+    </xacro:macro>
+    <!-- covers -->
+    <!-- shoulder_extension_ring -->
+    <xacro:macro name="shoulder_extension_ring" params="name xyz:=${triple_zero} rpy:=${triple_zero}">
+        <link name="${name}">
+            <inertial>
+                <origin xyz="${xyz}" rpy="${rpy}"/>
+                <mass value="0.01"/>
+                <inertia
+                    ixx="0.000008154" ixy="0" ixz="0"
+                    iyy="0.000007974" iyz="0.000000006"
+                    izz="0.000015238"
+                />
+            </inertial>
+            <visual>
+                <origin xyz="${xyz}" rpy="${rpy}"/>
+                <geometry>
+                    <mesh filename="package://separable_jaws_description/meshes/shoulder_extension_ring.stl"/>
+                </geometry>
+                <material name="${extension_ring_material}"/>
+            </visual>
+            <collision>
+                <origin xyz="${xyz}" rpy="${rpy}"/>
+                <geometry>
+                    <mesh filename="package://separable_jaws_description/meshes/shoulder_extension_ring.stl"/>
+                </geometry>
+            </collision>
+        </link>
+        <xacro:if value="$(arg using_gazebo)">
+            <gazebo reference="${name}">
+                <material>Gazebo/${extension_ring_material}</material>
+            </gazebo>
+        </xacro:if>
+    </xacro:macro>
+    <!-- shoulder_cover -->
+    <xacro:macro name="shoulder_cover" params="name xyz:=${triple_zero} rpy:=${triple_zero}">
+        <link name="${name}">
+            <inertial>
+                <origin xyz="${xyz}" rpy="${rpy}"/>
+                <mass value="0.075"/>
+                <inertia
+                    ixx="0.000055846" ixy="0" ixz="0"
+                    iyy="0.000055846" iyz="0"
+                    izz="0.000068514"
+                />
+            </inertial>
+            <visual>
+                <origin xyz="${xyz}" rpy="${rpy}"/>
+                <geometry>
+                    <mesh filename="package://separable_jaws_description/meshes/shoulder_cover.stl"/>
+                </geometry>
+                <material name="${cover_material}"/>
+            </visual>
+            <collision>
+                <origin xyz="${xyz}" rpy="${rpy}"/>
+                <geometry>
+                    <mesh filename="package://separable_jaws_description/meshes/shoulder_cover.stl"/>
+                </geometry>
+            </collision>
+        </link>
+        <xacro:if value="$(arg using_gazebo)">
+            <gazebo reference="${name}">
+                <material>Gazebo/${cover_material}</material>
+            </gazebo>
+        </xacro:if>
+    </xacro:macro>
+    <!-- upper_arm_cover -->
+    <xacro:macro name="upper_arm_cover" params="name xyz:=${triple_zero} rpy:=${triple_zero}">
+        <link name="${name}">
+            <inertial>
+                <origin xyz="${xyz}" rpy="${rpy}"/>
+                <mass value="0.235"/>
+                <inertia
+                    ixx="0.000385567" ixy="-0.00000002" ixz="0.000732197"
+                    iyy="0.006196229" iyz="-0.000000009"
+                    izz="0.00621496"
+                />
+            </inertial>
+            <visual>
+                <origin xyz="${xyz}" rpy="${rpy}"/>
+                <geometry>
+                    <mesh filename="package://separable_jaws_description/meshes/upper_arm_cover.stl"/>
+                </geometry>
+                <material name="${cover_material}"/>
+            </visual>
+            <collision>
+                <origin xyz="${xyz}" rpy="${rpy}"/>
+                <geometry>
+                    <mesh filename="package://separable_jaws_description/meshes/upper_arm_cover.stl"/>
+                </geometry>
+            </collision>
+        </link>
+        <xacro:if value="$(arg using_gazebo)">
+            <gazebo reference="${name}">
+                <material>Gazebo/${cover_material}</material>
+            </gazebo>
+        </xacro:if>
+    </xacro:macro>
+    <!-- lower_arm_cover -->
+    <xacro:macro name="lower_arm_cover" params="name xyz:=${triple_zero} rpy:=${triple_zero}">
+        <link name="${name}">
+            <inertial>
+                <origin xyz="${xyz}" rpy="${rpy}"/>
+                <mass value="0.079"/>
+                <inertia
+                    ixx="0.000047626" ixy="0.000000367" ixz="0.000039299"
+                    iyy="0.001178645" iyz="-0.000000021"
+                    izz="0.00121964"
+                />
+            </inertial>
+            <visual>
+                <origin xyz="${xyz}" rpy="${rpy}"/>
+                <geometry>
+                    <mesh filename="package://separable_jaws_description/meshes/lower_arm_cover.stl"/>
+                </geometry>
+                <material name="${cover_material}"/>
+            </visual>
+            <collision>
+                <origin xyz="${xyz}" rpy="${rpy}"/>
+                <geometry>
+                    <mesh filename="package://separable_jaws_description/meshes/lower_arm_cover.stl"/>
+                </geometry>
+            </collision>
+        </link>
+        <xacro:if value="$(arg using_gazebo)">
+            <gazebo reference="${name}">
+                <material>Gazebo/${cover_material}</material>
+            </gazebo>
+        </xacro:if>
+    </xacro:macro>
+    <!-- wrist_extension_ring -->
+    <xacro:macro name="wrist_extension_ring" params="name xyz:=${triple_zero} rpy:=${triple_zero}">
+        <link name="${name}">
+            <inertial>
+                <origin xyz="${xyz}" rpy="${rpy}"/>
+                <mass value="0.007"/>
+                <inertia
+                    ixx="0.000003276" ixy="0" ixz="0"
+                    iyy="0.000003197" iyz="0.000000003"
+                    izz="0.00000617"
+                />
+            </inertial>
+            <visual>
+                <origin xyz="${xyz}" rpy="${rpy}"/>
+                <geometry>
+                    <mesh filename="package://separable_jaws_description/meshes/wrist_extension_ring.stl"/>
+                </geometry>
+                <material name="${extension_ring_material}"/>
+            </visual>
+            <collision>
+                <origin xyz="${xyz}" rpy="${rpy}"/>
+                <geometry>
+                    <mesh filename="package://separable_jaws_description/meshes/wrist_extension_ring.stl"/>
+                </geometry>
+            </collision>
+        </link>
+        <xacro:if value="$(arg using_gazebo)">
+            <gazebo reference="${name}">
+                <material>Gazebo/${extension_ring_material}</material>
+            </gazebo>
+        </xacro:if>
+    </xacro:macro>
+    <!-- wrist_cover -->
+    <xacro:macro name="wrist_cover" params="name xyz:=${triple_zero} rpy:=${triple_zero}">
+        <link name="${name}">
+            <inertial>
+                <origin xyz="${xyz}" rpy="${rpy}"/>
+                <mass value="0.037"/>
+                <inertia
+                    ixx="0.000009686" ixy="0" ixz="0"
+                    iyy="0.00000987" iyz="0"
+                    izz="0.000017485"
+                />
+            </inertial>
+            <visual>
+                <origin xyz="${xyz}" rpy="${rpy}"/>
+                <geometry>
+                    <mesh filename="package://separable_jaws_description/meshes/wrist_cover.stl"/>
+                </geometry>
+                <material name="${cover_material}"/>
+            </visual>
+            <collision>
+                <origin xyz="${xyz}" rpy="${rpy}"/>
+                <geometry>
+                    <mesh filename="package://separable_jaws_description/meshes/wrist_cover.stl"/>
+                </geometry>
+            </collision>
+        </link>
+        <xacro:if value="$(arg using_gazebo)">
+            <gazebo reference="${name}">
+                <material>Gazebo/${cover_material}</material>
+            </gazebo>
+        </xacro:if>
     </xacro:macro>
     <!-- motors -->
@@ -184,7 +389,9 @@
             </collision>
         </link>
-        <gazebo reference="${name}">
-            <material>Gazebo/${motor_material}</material>
-        </gazebo>
+        <xacro:if value="$(arg using_gazebo)">
+            <gazebo reference="${name}">
+                <material>Gazebo/${motor_material}</material>
+            </gazebo>
+        </xacro:if>
     </xacro:macro>
     <!-- dynamixel_pro_h54-200-s500 -->
@@ -214,7 +421,9 @@
             </collision>
         </link>
-        <gazebo reference="${name}">
-            <material>Gazebo/${motor_material}</material>
-        </gazebo>
+        <xacro:if value="$(arg using_gazebo)">
+            <gazebo reference="${name}">
+                <material>Gazebo/${motor_material}</material>
+            </gazebo>
+        </xacro:if>
     </xacro:macro>
     <!-- dynamixel_pro_h42-20-s300-->
@@ -244,7 +453,9 @@
             </collision>
         </link>
-        <gazebo reference="${name}">
-            <material>Gazebo/${motor_material}</material>
-        </gazebo>
+        <xacro:if value="$(arg using_gazebo)">
+            <gazebo reference="${name}">
+                <material>Gazebo/${motor_material}</material>
+            </gazebo>
+        </xacro:if>
     </xacro:macro>
 </robot>

File: urdf/separable_jaws.xacro (robot description, xacro)
@@ -1,16 +1,30 @@
 <?xml version="1.0"?>
 <robot name="separable_jaws" xmlns:xacro="http://www.ros.org/wiki/xacro">
+    <!-- declare arguments -->
+    <xacro:arg name="using_left_arm" default="true"/>
+    <xacro:arg name="using_right_arm" default="true"/>
+    <xacro:arg name="using_gazebo" default="false"/>
+    <xacro:arg name="using_fake_hardware" default="true"/>
     <!-- include macros from other files-->
     <xacro:include filename="$(find separable_jaws_description)/urdf/material.xacro"/>
-    <xacro:include filename="$(find separable_jaws_description)/urdf/simple_geometry.xacro"/>
     <xacro:include filename="$(find separable_jaws_description)/urdf/parts.xacro"/>
     <xacro:include filename="$(find separable_jaws_description)/urdf/subassemblies.xacro"/>
     <!-- robot definition -->
     <link name="base_link"/>
-    <xacro:right_bracket xyz="0 0 1"/>
-    <xacro:right_shoulder/>
-    <xacro:right_upper_arm/>
-    <xacro:right_lower_arm/>
-    <xacro:right_wrist/>
-    <xacro:right_palm/>
+    <xacro:if value="$(arg using_left_arm)">
+        <xacro:left_bracket xyz="0 0.05 0.2"/>
+        <xacro:left_shoulder/>
+        <xacro:left_upper_arm/>
+        <xacro:left_lower_arm/>
+        <xacro:left_wrist/>
+        <xacro:left_palm/>
+    </xacro:if>
+    <xacro:if value="$(arg using_right_arm)">
+        <xacro:right_bracket xyz="0 -0.05 0.2"/>
+        <xacro:right_shoulder/>
+        <xacro:right_upper_arm/>
+        <xacro:right_lower_arm/>
+        <xacro:right_wrist/>
+        <xacro:right_palm/>
+    </xacro:if>
 </robot>
