Commit message: fix dependencies

File: urdf/subassemblies.xacro (robot description, xacro)
@@ -22,5 +22,5 @@
         <xacro:shoulder_extension_ring name="left_shoulder_extension_ring"/>
         <xacro:shoulder_cover name="left_shoulder_cover"/>
-        <joint name="left_shoulder_joint" type="revolute">
+        <joint name="left_shoulder_joint" type="continuous">
             <origin xyz="0 -0.025 0" rpy="0 ${radians(180)} 0"/>
             <parent link="left_bracket"/>
@@ -51,5 +51,5 @@
         <xacro:upper_arm_cover name="left_upper_arm_cover"/>
         <xacro:dynamixel_pro_h54-100-s500 name="left_upper_arm_motor2" rpy="0 ${radians(90)} ${radians(90)}"/>
-        <joint name="left_upper_arm_joint" type="revolute">
+        <joint name="left_upper_arm_joint" type="continuous">
             <origin xyz="0.045 -0.0505 0" rpy="${radians(-90)} 0 0"/>
             <parent link="left_shoulder"/>
@@ -79,5 +79,5 @@
         <xacro:lower_arm_cover name="left_lower_arm_cover"/>
         <xacro:dynamixel_pro_h42-20-s300 name="left_lower_arm_motor" rpy="0 0 ${radians(-90)}"/>
-        <joint name="left_lower_arm_joint" type="revolute">
+        <joint name="left_lower_arm_joint" type="continuous">
             <origin xyz="0 0 0" rpy="0 0 0"/>
             <parent link="left_upper_arm_motor2"/>
@@ -103,5 +103,5 @@
         <xacro:wrist_cover name="left_wrist_cover"/>
         <xacro:dynamixel_pro_h42-20-s300 name="left_wrist_motor" rpy="0 ${radians(-90)} ${radians(180)}"/>
-        <joint name="left_wrist_joint" type="revolute">
+        <joint name="left_wrist_joint" type="continuous">
             <origin xyz="0 0 0" rpy="${radians(-90)} 0 0"/>
             <parent link="left_lower_arm_motor"/>
@@ -132,5 +132,5 @@
         <xacro:wrist_cover name="left_palm_cover"/>
         <xacro:dynamixel_pro_h42-20-s300 name="left_palm_motor" rpy="0 ${radians(-90)} ${radians(180)}"/>
-        <joint name="left_palm_joint" type="revolute">
+        <joint name="left_palm_joint" type="continuous">
             <origin xyz="0 0 0" rpy="0 ${radians(180)} ${radians(90)}"/>
             <parent link="left_wrist_motor"/>
@@ -170,5 +170,5 @@
         <xacro:shoulder_extension_ring name="right_shoulder_extension_ring"/>
         <xacro:shoulder_cover name="right_shoulder_cover"/>
-        <joint name="right_shoulder_joint" type="revolute">
+        <joint name="right_shoulder_joint" type="continuous">
             <origin xyz="0 -0.025 0" rpy="0 0 0"/>
             <parent link="right_bracket"/>
@@ -199,5 +199,5 @@
         <xacro:upper_arm_cover name="right_upper_arm_cover"/>
         <xacro:dynamixel_pro_h54-100-s500 name="right_upper_arm_motor2" rpy="0 ${radians(90)} ${radians(90)}"/>
-        <joint name="right_upper_arm_joint" type="revolute">
+        <joint name="right_upper_arm_joint" type="continuous">
             <origin xyz="0.045 -0.0505 0" rpy="${radians(90)} 0 0"/>
             <parent link="right_shoulder"/>
@@ -227,5 +227,5 @@
         <xacro:lower_arm_cover name="right_lower_arm_cover"/>
         <xacro:dynamixel_pro_h42-20-s300 name="right_lower_arm_motor" rpy="0 ${radians(180)} ${radians(-90)}"/>
-        <joint name="right_lower_arm_joint" type="revolute">
+        <joint name="right_lower_arm_joint" type="continuous">
             <origin xyz="0 0 0" rpy="0 0 0"/>
             <parent link="right_upper_arm_motor2"/>
@@ -251,5 +251,5 @@
         <xacro:wrist_cover name="right_wrist_cover"/>
         <xacro:dynamixel_pro_h42-20-s300 name="right_wrist_motor" rpy="0 ${radians(-90)} ${radians(180)}"/>
-        <joint name="right_wrist_joint" type="revolute">
+        <joint name="right_wrist_joint" type="continuous">
             <origin xyz="0 0 0" rpy="${radians(90)} 0 0"/>
             <parent link="right_lower_arm_motor"/>
@@ -280,5 +280,5 @@
         <xacro:wrist_cover name="right_palm_cover"/>
         <xacro:dynamixel_pro_h42-20-s300 name="right_palm_motor" rpy="0 ${radians(-90)} ${radians(180)}"/>
-        <joint name="right_palm_joint" type="revolute">
+        <joint name="right_palm_joint" type="continuous">
             <origin xyz="0 0 0" rpy="0 ${radians(180)} ${radians(90)}"/>
             <parent link="right_wrist_motor"/>
